File: kicad/ps28-modern.kicad_pcb (KiCad board)
At the start: 4 copper layers, 0 parts

Commit message: baby steps
Parts:
- added C10: 1uF 100V X7R, Capacitor_SMD:C_1206_3216Metric, F.Cu at (84.0, 55.0)
- added C11: 1uF 100V X7R, Capacitor_SMD:C_1206_3216Metric, F.Cu at (84.0, 60.0)
- added C12: 1uF 100V X7R, Capacitor_SMD:C_1206_3216Metric, F.Cu at (84.0, 65.0)
- added C13: 1uF 100V X7R, Capacitor_SMD:C_1206_3216Metric, F.Cu at (84.0, 70.0)
- added C16: 33nF 25V X7R, Capacitor_SMD:C_0603_1608Metric, F.Cu at (85.0, 48.0)
- added C17: 33nF 25V X7R, Capacitor_SMD:C_0603_1608Metric, F.Cu at (89.0, 57.0)
- added C18: 33nF 25V X7R, Capacitor_SMD:C_0603_1608Metric, F.Cu at (89.0, 66.0)
- added C19: 33nF 25V X7R, Capacitor_SMD:C_0603_1608Metric, F.Cu at (85.0, 77.0)
- added C2: 100nF 25V X7R, Capacitor_SMD:C_0603_1608Metric, F.Cu at (66.0, 52.0)
- added C20: 10uF 16V X7R, Capacitor_SMD:C_1206_3216Metric, F.Cu at (55.0, 46.0)
- added C21: 10uF 16V X7R, Capacitor_SMD:C_1206_3216Metric, F.Cu at (55.0, 50.0)
- added C24: 1nF 100V C0G, Capacitor_SMD:C_0603_1608Metric, F.Cu at (139.0, 45.0)
- added C25: 10nF 100V dielectric TBD, Capacitor_SMD:C_1206_3216Metric, F.Cu at (144.0, 45.0)
- added C28: 1nF 100V C0G, Capacitor_SMD:C_0603_1608Metric, F.Cu at (139.0, 80.0)
- added C29: 10nF 100V dielectric TBD, Capacitor_SMD:C_1206_3216Metric, F.Cu at (144.0, 80.0)
- added C3: 10uF 25V X7R, Capacitor_SMD:C_1206_3216Metric, F.Cu at (61.0, 52.0)
- added C4: 100nF 25V X7R, Capacitor_SMD:C_0603_1608Metric, F.Cu at (65.0, 56.0)
- added C5: 100nF 25V X7R, Capacitor_SMD:C_0603_1608Metric, F.Cu at (65.0, 69.0)
- added C6: 1uF 16V X7R, Capacitor_SMD:C_0603_1608Metric, F.Cu at (61.0, 60.0)
- added C7: 1uF 16V X7R, Capacitor_SMD:C_0603_1608Metric, F.Cu at (56.0, 56.0)
- added C8: 47nF 25V X7R, Capacitor_SMD:C_0603_1608Metric, F.Cu at (56.0, 60.0)
- added C9: 1uF 16V X7R, Capacitor_SMD:C_0603_1608Metric, F.Cu at (60.0, 72.0)
- added J2: 12V auxiliary, Connector_PinHeader_2.54mm:PinHeader_1x02_P2.54mm_Vertical, F.Cu at (35.0, 35.0)
- added J3: Differential audio interface, Connector_PinHeader_2.54mm:PinHeader_1x03_P2.54mm_Vertical, F.Cu at (35.0, 65.0)
- added J4: Control: 3V3 RESET FAULT CLIP GND, Connector_PinHeader_2.54mm:PinHeader_1x05_P2.54mm_Vertical, F.Cu at (35.0, 85.0)
- added R1: 3.3R, Resistor_SMD:R_0603_1608Metric, F.Cu at (64.0, 48.0)
- added R2: 3.3R, Resistor_SMD:R_0603_1608Metric, F.Cu at (64.0, 73.0)
- added R3: 22k 1%, Resistor_SMD:R_0603_1608Metric, F.Cu at (55.0, 64.0)
- added R4: 30k 1%, Resistor_SMD:R_0603_1608Metric, F.Cu at (55.0, 68.0)
- added R5: 3.3R power TBD, Resistor_SMD:R_1206_3216Metric, F.Cu at (144.0, 50.0)
- added R6: 3.3R power TBD, Resistor_SMD:R_1206_3216Metric, F.Cu at (144.0, 85.0)
- added R7: 10k, Resistor_SMD:R_0603_1608Metric, F.Cu at (40.0, 90.0)
- added R8: 10k, Resistor_SMD:R_0603_1608Metric, F.Cu at (40.0, 94.0)
- added R9: 10k RESET safe-low, Resistor_SMD:R_0603_1608Metric, F.Cu at (40.0, 98.0)
- added U1: TPA3255DDV, Package_SO:HTSSOP-44_6.1x14mm_P0.635mm_TopEP4.14x7.01mm, F.Cu at (75.0, 60.0)
Other:
- board outline added: 145 x 95 mm
- board text added: "145 x 95 mm provisional outline; NOT a measured mechanical envelope"
- board text added: "L1 reservation only - MPN/pads TBD"
- board text added: "L2 reservation only - MPN/pads TBD"
- board text added: "PVDD bulk + connector reservation"
- board text added: "TOP HEATSINK: envelope/bond/fixing TBD"
- board text added: "UNROUTED CORE ONLY - NOT FOR FABRICATION"
