File: kicad/ps28-modern.kicad_sch (KiCad schematic)
At the start: 0 parts

Commit message: baby steps
Parts:
- added C1: 470uF voltage/ripple TBD, symbol Device:C_Polarized
- added C10, C11, C12, C13: 1uF 100V X7R, Capacitor_SMD:C_1206_3216Metric, symbol Device:C
- added C14, C15: 470uF 63V ripple TBD, symbol Device:C_Polarized
- added C16, C17, C18, C19: 33nF 25V X7R, Capacitor_SMD:C_0603_1608Metric, symbol Device:C
- added C2, C4, C5: 100nF 25V X7R, Capacitor_SMD:C_0603_1608Metric, symbol Device:C
- added C20, C21: 10uF 16V X7R, Capacitor_SMD:C_1206_3216Metric, symbol Device:C
- added C22, C23, C26, C27: 470nF 100V dielectric TBD, symbol Device:C
- added C24, C28: 1nF 100V C0G, Capacitor_SMD:C_0603_1608Metric, symbol Device:C
- added C25, C29: 10nF 100V dielectric TBD, Capacitor_SMD:C_1206_3216Metric, symbol Device:C
- added C3: 10uF 25V X7R, Capacitor_SMD:C_1206_3216Metric, symbol Device:C
- added C6, C7, C9: 1uF 16V X7R, Capacitor_SMD:C_0603_1608Metric, symbol Device:C
- added C8: 47nF 25V X7R, Capacitor_SMD:C_0603_1608Metric, symbol Device:C
- added J1: 36V regulated input - connector TBD, symbol Connector_Generic:Conn_01x02
- added J2: 12V auxiliary, Connector_PinHeader_2.54mm:PinHeader_1x02_P2.54mm_Vertical, symbol Connector_Generic:Conn_01x02
- added J3: Differential audio interface, Connector_PinHeader_2.54mm:PinHeader_1x03_P2.54mm_Vertical, symbol Connector_Generic:Conn_01x03
- added J4: Control: 3V3 RESET FAULT CLIP GND, Connector_PinHeader_2.54mm:PinHeader_1x05_P2.54mm_Vertical, symbol Connector_Generic:Conn_01x05
- added J5: Floating speaker - connector TBD, symbol Connector_Generic:Conn_01x02
- added J6: Grounded top heatsink bond - mechanical TBD, symbol Connector_Generic:Conn_01x01
- added L1, L2: 10uH Isat/Irms/MPN TBD, symbol Device:L
- added R1, R2: 3.3R, Resistor_SMD:R_0603_1608Metric, symbol Device:R
- added R3: 22k 1%, Resistor_SMD:R_0603_1608Metric, symbol Device:R
- added R4: 30k 1%, Resistor_SMD:R_0603_1608Metric, symbol Device:R
- added R5, R6: 3.3R power TBD, Resistor_SMD:R_1206_3216Metric, symbol Device:R
- added R7, R8: 10k, Resistor_SMD:R_0603_1608Metric, symbol Device:R
- added R9: 10k RESET safe-low, Resistor_SMD:R_0603_1608Metric, symbol Device:R
- added U1: TPA3255DDV, Package_SO:HTSSOP-44_6.1x14mm_P0.635mm_TopEP4.14x7.01mm, symbol PS28:TPA3255DDV
Connections:
- new net AUX_12V: C1.1, C2.1, C3.1, J2.1 (Pin_1), R1.1, R2.1, U1.2 (VDD)
- new net AVDD: C7.1, U1.14 (AVDD)
- new net BST_A: C16.1, U1.44 (BST_A)
- new net BST_B: C17.1, U1.43 (BST_B)
- new net BST_C: C18.1, U1.24 (BST_C)
- new net BST_D: C19.1, U1.23 (BST_D)
- new net CLIP_OTW: J4.4 (Pin_4), R8.2, U1.21 (~{CLIP_OTW})
- new net C_START: C8.1, U1.15 (C_START)
- new net DIFF_N: C21.1, J3.2 (Pin_2)
- new net DIFF_P: C20.1, J3.1 (Pin_1)
- new net DVDD_INTERNAL: C6.1, U1.11 (DVDD), U1.4 (M2)
- new net FAULT: J4.3 (Pin_3), R7.2, U1.19 (~{FAULT})
- new net FREQ_ADJ: R4.1, U1.8 (FREQ_ADJ)
- new net GND: C1.2, C10.2, C11.2, C12.2, C13.2, C14.2, C15.2, C2.2, C22.2, C23.2, C24.2, C26.2, C27.2, C28.2, C3.2, C4.2, C5.2, C6.2, C7.2, C8.2, C9.2, J1.2 (Pin_2), J2.2 (Pin_2), J3.3 (Pin_3), J4.5 (Pin_5), J6.1 (Pin_1), R3.2, R4.2, R5.2, R6.2, R9.2, U1.12 (GND), U1.13 (GND), U1.16 (INPUT_C), U1.17 (INPUT_D), U1.25 (GND), U1.26 (GND), U1.3 (M1), U1.33 (GND), U1.34 (GND), U1.41 (GND), U1.42 (GND)
- new net GVDD_AB: C4.1, R1.2, U1.1 (GVDD_AB)
- new net GVDD_CD: C5.1, R2.2, U1.22 (GVDD_CD)
- new net INPUT_A_AC: C20.2, U1.5 (INPUT_A)
- new net INPUT_B_AC: C21.2, U1.6 (INPUT_B)
- new net OC_ADJ: R3.1, U1.7 (OC_ADJ)
- new net PVDD_36V: C10.1, C11.1, C12.1, C13.1, C14.1, C15.1, J1.1 (Pin_1), U1.29 (PVDD_CD), U1.30 (PVDD_CD), U1.31 (PVDD_CD), U1.36 (PVDD_AB), U1.37 (PVDD_AB), U1.38 (PVDD_AB)
- new net PWM_AC: C16.2, C18.2, L1.1, U1.32 (OUT_C), U1.39 (OUT_A), U1.40 (OUT_A)
- new net PWM_BD: C17.2, C19.2, L2.1, U1.27 (OUT_D), U1.28 (OUT_D), U1.35 (OUT_B)
- new net RESET: J4.2 (Pin_2), R9.1, U1.18 (~{RESET})
- new net SPK_N: C26.1, C27.1, C28.1, C29.1, J5.2 (Pin_2), L2.2
- new net SPK_N_SNUB: C29.2, R6.1
- new net SPK_P: C22.1, C23.1, C24.1, C25.1, J5.1 (Pin_1), L1.2
- new net SPK_P_SNUB: C25.2, R5.1
- new net VBG: C9.1, U1.20 (VBG)
- new net VIO_3V3_EXTERNAL: J4.1 (Pin_1), R7.1, R8.1
- no-connect marks 0 -> 2
Other:
- note added: "CORE ONLY - RESET DEFAULT LOW - NO SUPPLY/FRONT-END - NO MANUFACTURING"
- title: PS28 Modern Amp - EMPTY CONTAINER -> PS28 - TPA3255 CORE DRAFT - NOT FOR FABRICATION
