File: kicad/seq-d020/seq-d020.kicad_sch (KiCad schematic)
At the start: 48 parts, among them J401 START_BUTTON, J402 SEQ_TO_SYSTEM, U401 LP2985-33, U402 TPS3808G33, U403 TPS3808G33, U404 TPS3808G33, U405 74LVC1G14, U406 74LVC2G74, U407 74LVC2G74, U408 74LVC1G32, U409 74LVC1G07, U410 74LVC1G08, U411 74LVC1G06, U412 TPS3700DDC, U413 TPS3700DDC

Commit message: feat(eda): complete D-019 input interface with Form C relay, mute and DC observation
- iso-d019 (D-024): Omron G6K-2F DC12 after C20/C21 (COM isolated plate,
  NO TPA pin, NC 1k discharge; break-before-make, isolated when unpowered),
  TMUX6219 mute DIVIDED->VMID, TPS3700 DC windows on both pins (2-5 V,
  tau ~50 ms) and AUX_RAW window, MMBT3904 relay/mute drivers.
- seq-d020: RESET released 12-28 ms after relay command, DC dwell 12-28 ms
  before AUDIO_EN latch, DC loss trips RAILS_OK, start timeout covers dwell.
- simulate_d019: 1350 ngspice cases, pin -0.262..6.61 V within -0.3..7 V
  (worst with pessimistic 10 ms opening; >= 0 V at datasheet 3 ms).
- system-candidate: 200 footprints, 570 pins matched, bridge closed only
  via K501, J3 DNP; ERC equal to base, DRC 0, 464 unrouted.
- Not covered: single-fault preamp rail/driver short, real TPA input when
  unpowered, contact bounce/stuck, content below 20 Hz.
Parts:
- added C418, C419, C420, C421, C422, C423: 100n, Capacitor_SMD:C_0603_1608Metric, symbol Device:C
- added R428, R429, R430: 100k, Resistor_SMD:R_0603_1608Metric, symbol Device:R
- added U414, U416: TPS3808G33, Package_TO_SOT_SMD:SOT-23-6, symbol Power_Supervisor:TPS3808DBV
- added U415: 74LVC1G08, Package_TO_SOT_SMD:SOT-23-5, symbol 74xGxx:74LVC1G08
- added U417: 74LVC2G74, Package_SO:SSOP-8_2.95x2.8mm_P0.65mm, symbol 74xGxx:74LVC2G74
- added U418: 74LVC1G32, Package_TO_SOT_SMD:SOT-23-5, symbol 74xGxx:74LVC1G32
- added U419: 74LVC1G07, Package_TO_SOT_SMD:SOT-23-5, symbol 74xGxx:74LVC1G07
- J402: symbol Connector_Generic:Conn_01x07 -> Connector_Generic:Conn_01x10; MPN Logical interface to power-d021/core; same PCB, not a conne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 -> Logical interface to power-d021/iso-d019/core; same PCB, no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
Connections:
- net GND: now also C418.2, C419.2, C420.2, C421.2, C422.2, C423.2, U414.2 (GND), U415.3 (GND), U416.2 (GND), U417.4 (GND), U418.3 (GND), U419.3 (GND)
- net NOT_ARMED: no longer U410.2
- net RAILS_OK: now also U419.4
- net RUN: now also J402.8 (Pin_8), U414.3 (~{MR}), U417.6 (~{CLR}); no longer R408.1
- net SEQ_3V3: now also C418.1, C419.1, C420.1, C421.1, C422.1, C423.1, R428.1, R429.1, R430.1, U414.5 (SENSE), U414.6 (VDD), U415.5 (VCC), U416.5 (SENSE), U416.6 (VDD), U417.2 (D), U417.7 (~{PRE}), U417.8 (VCC), U418.5 (VCC), U419.5 (VCC)
- net ARMED: now reaches U407.5 (Q)
- net ARMED: now also U415.1
- new net AUDIO_EN: J402.9 (Pin_9), U417.5 (Q)
- new net DC_GATE: U415.4, U416.3 (~{MR})
- new net DC_OK: J402.10 (Pin_10), R429.2, U415.2, U418.2
- new net DC_TRIP_N: U418.4, U419.2
- new net DWELL_OK: R430.2, U416.1 (~{RESET}), U417.1 (C)
- new net NOT_AUDIO: U410.2, U417.3 (~{Q}), U418.1
- new net RESET_GO: R408.1, R428.2, U414.1 (~{RESET})
- no-connect marks 4 -> 6
Other:
- note added: "RELAY/MUTE/DC WINDOWS IN iso-d019. FOOTPRINTS NOT AUDITED. DO NOT ENERGIZE."
- note removed: "NO INPUT ISOLATION/DISCHARGE/DC SENSE/MUTE (D-019 OPEN). FOOTPRINTS NOT AUDITED. DO NOT ENERGIZE."
- moved on the sheet: C406, C407, C408, C409, C410, C411, C412, C413, C414, C415, C416, C417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
